File: Schematic/Embedded.sch (EAGLE design)
At the start: 20 parts, among them T1 2N3904, T2 2N3904, T3 2N3904, T4 2N3904

Commit message: Added Relay Definitions
Parts:
- removed PB: SSW-110-02-G-S, con-samtec:SSW-110-02-G-S
- removed PHSENSOR: SSW-104-02-G-S, con-samtec:SSW-104-02-G-S
- added JP1: (no value), pinhead:PINHD-1X3
Connections:
- removed net N$18: PHSENSOR-1.1
- removed net N$20: PHSENSOR-2.1
- removed net N$21: PHSENSOR-3.1
- removed net N$22: PHSENSOR-4.1
- net +5V: now also JP1.2
- net A0: now also JP1.3
- net D4: now also R2.1; no longer R3.2
- net GND: now also JP1.1
- net N$1: now also R2.2; no longer R3.1
- net N$7: now also R3.2; no longer R2.1
- net N$9: now also R3.1; no longer R2.2
Other:
- moved on the sheet: PD-1, PD-2, PD-3, PD-4, PD-5, PD-6, PD-7, PD-8, R2, R3

Commit message: I believe that I finally Finished.
Parts:
- R2: value 1k -> 10k
- R3: value 10k -> 1k
Connections:
- removed net N$14: R5.2
- removed net N$19: R7.2
- removed net N$9: R3.1
- new net 5V: R3.1, R5.2, R7.2

Commit message: Fixed Disconnected 5V
Connections:
- removed net 5V: R3.1, R5.2, R7.2
- net +5V: now also R3.1, R5.2, R7.2
Changed lines of the file:
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@@
 <part name="P+9" library="supply1" library_urn="urn:adsk.eagle:library:371" deviceset="+5V" device=""/>
 <part name="SUPPLY9" library="supply2" library_urn="urn:adsk.eagle:library:372" deviceset="GND" device=""/>
+<part name="P+4" library="supply1" library_urn="urn:adsk.eagle:library:371" deviceset="+5V" device=""/>
+<part name="P+5" library="supply1" library_urn="urn:adsk.eagle:library:371" deviceset="+5V" device=""/>
+<part name="P+6" library="supply1" library_urn="urn:adsk.eagle:library:371" deviceset="+5V" device=""/>
 </parts>
 <sheets>
@@
 <attribute name="VALUE" x="150.495" y="73.025" size="1.778" layer="96"/>
 </instance>
+<instance part="P+4" gate="1" x="111.76" y="48.26" smashed="yes" rot="R180">
+<attribute name="VALUE" x="114.3" y="53.34" size="1.778" layer="96" rot="R270"/>
+</instance>
+<instance part="P+5" gate="1" x="165.1" y="48.26" smashed="yes" rot="R180">
+<attribute name="VALUE" x="167.64" y="53.34" size="1.778" layer="96" rot="R270"/>
+</instance>
+<instance part="P+6" gate="1" x="208.28" y="48.26" smashed="yes" rot="R180">
+<attribute name="VALUE" x="210.82" y="53.34" size="1.778" layer="96" rot="R270"/>
+</instance>
 </instances>
 <busses>
@@
 <wire x1="124.46" y1="76.2" x2="124.46" y2="78.74" width="0.1524" layer="91"/>
 </segment>
+<segment>
+<pinref part="P+4" gate="1" pin="+5V"/>
+<wire x1="111.76" y1="50.8" x2="111.76" y2="55.88" width="0.1524" layer="91"/>
+<pinref part="R3" gate="G$1" pin="1"/>
+<wire x1="104.14" y1="55.88" x2="111.76" y2="55.88" width="0.1524" layer="91"/>
+<label x="106.68" y="55.88" size="1.778" layer="95"/>
+</segment>
+<segment>
+<pinref part="P+5" gate="1" pin="+5V"/>
+<wire x1="165.1" y1="50.8" x2="165.1" y2="55.88" width="0.1524" layer="91"/>
+<pinref part="R5" gate="G$1" pin="2"/>
+<wire x1="157.48" y1="55.88" x2="165.1" y2="55.88" width="0.1524" layer="91"/>
+<label x="160.02" y="55.88" size="1.778" layer="95"/>
+</segment>
+<segment>
+<pinref part="P+6" gate="1" pin="+5V"/>
+<wire x1="208.28" y1="50.8" x2="208.28" y2="55.88" width="0.1524" layer="91"/>
+<pinref part="R7" gate="G$1" pin="2"/>
+<wire x1="200.66" y1="55.88" x2="208.28" y2="55.88" width="0.1524" layer="91"/>
+<label x="203.2" y="55.88" size="1.778" layer="95"/>
+</segment>
 </net>
 <net name="GND" class="0">
@@
 </segment>
 </net>
-<net name="5V" class="0">
-<segment>
-<pinref part="R3" gate="G$1" pin="1"/>
-<wire x1="104.14" y1="55.88" x2="111.76" y2="55.88" width="0.1524" layer="91"/>
-<label x="106.68" y="55.88" size="1.778" layer="95"/>
-</segment>
-<segment>
-<pinref part="R5" gate="G$1" pin="2"/>
-<wire x1="157.48" y1="55.88" x2="165.1" y2="55.88" width="0.1524" layer="91"/>
-<label x="160.02" y="55.88" size="1.778" layer="95"/>
-</segment>
-<segment>
-<pinref part="R7" gate="G$1" pin="2"/>
-<wire x1="200.66" y1="55.88" x2="208.28" y2="55.88" width="0.1524" layer="91"/>
-<label x="203.2" y="55.88" size="1.778" layer="95"/>
-</segment>
-</net>

Commit message: Checked Wires
Found a GND wire that is thin to a point. Unfortunately, the PCB is already  printed.
Parts:
- added X1: TSW-108-07-G-S, con-samtec:TSW-108-07-G-S
Connections:
- new net P1: T1.E, X1-1.1
- new net P2: T2.E, X1-3.1
- new net P3: T3.E, X1-5.1
- new net P4: T4.E, X1-7.1
- net +5V: now also UTILITY-5.1; no longer UTILITY-6.1
- net GND: now also UTILITY-6.1, X1-2.1, X1-4.1, X1-6.1, X1-8.1; no longer T1.E, T2.E, T3.E, T4.E
Other:
- moved on the sheet: PC-1, PC-2, PC-3, PC-4, PC-5, PC-6
